File: piezo_signal_conditioner/piezo_signal_conditioner.kicad_sch (KiCad schematic)
At the start: 13 parts, among them U1 MCP6002-xP

Commit message: working proof of concept on breadboard
Parts:
- removed piezo_sensor: C, symbol Device:C
- added C3: piezo, symbol Device:C_Polarized
- added J1: input from drum, symbol Connector:Conn_01x02_Pin
- added J2: Conn_01x02_Pin, symbol Connector:Conn_01x02_Pin
- added R6: 120k, symbol Device:R
- added R7: 150k, symbol Device:R
- R5: value 100k -> 265k
Connections:
- net GND: now also J1.2 (Pin_2)
- net at R1.1, R2.1: now also J1.1 (Pin_1)
- new net: C3.1, R6.1
- new net: C3.2, J2.2 (Pin_2), R7.2
- new net: J2.1 (Pin_1), R6.2, R7.1
Other:
- note added: "Alesis Drum"

Commit message: circuit working
Parts:
- R5: value 265k -> 270k
- R6: value 120k -> 100k
Connections:
- net at R6.1: now also C3.2; no longer C3.1
- net negative output: now reaches J2.2 (Pin_2), R7.2
- net negative output: now also C3.1; no longer C3.2
- net positive output: now reaches J2.1 (Pin_1), R6.2, R7.1
Changed lines of the file:
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@@
+		)
+	)
+	(global_label "positive output"
+		(shape input)
+		(at 77.47 133.35 0)
+		(fields_autoplaced yes)
+		(effects
+			(font
+				(size 1.27 1.27)
+			)
+			(justify left)
+		)
+		(property "Intersheetrefs" "${INTERSHEET_REFS}"
+			(at 94.7878 133.35 0)
+			(effects
+				(font
+					(size 1.27 1.27)
+				)
+				(justify left)
+				(hide yes)
+			)
+		)
+	)
+	(global_label "negative output"
+		(shape input)
+		(at 77.47 148.59 0)
+		(fields_autoplaced yes)
+		(effects
+			(font
+				(size 1.27 1.27)
+			)
+			(justify left)
+		)
+		(property "Intersheetrefs" "${INTERSHEET_REFS}"
+			(at 95.3925 148.59 0)
+			(effects
+				(font
+					(size 1.27 1.27)
+				)
+				(justify left)
+				(hide yes)
+			)
 		)
 	)
@@
 			)
 		)
-		(property "Value" "265k"
+		(property "Value" "270k"
 			(at 180.34 73.6599 0)
 			(effects
@@
 		(lib_id "Device:C_Polarized")
 		(at 41.91 140.97 0)
-		(unit 1)
-		(exclude_from_sim no)
-		(in_bom yes)
-		(on_board yes)
-		(dnp no)
-		(fields_autoplaced yes)
+		(mirror x)
+		(unit 1)
+		(exclude_from_sim no)
+		(in_bom yes)
+		(on_board yes)
+		(dnp no)
 		(property "Reference" "C3"
-			(at 45.72 138.8109 0)
+			(at 45.72 143.1291 0)
 			(effects
 				(font
@@
 		)
 		(property "Value" "piezo"
-			(at 45.72 141.3509 0)
+			(at 45.72 140.5891 0)
 			(effects
 				(font
@@
 		)
 		(property "Footprint" ""
-			(at 42.8752 144.78 0)
+			(at 42.8752 137.16 0)
 			(effects
 				(font
@@
 			)
 		)
-		(property "Value" "120k"
+		(property "Value" "100k"
 			(at 54.61 129.54 90)
 			(effects

Commit message: changed discharge resistor to 100k for more reliable triggering
Parts:
- R5: value 270k -> 100k
Changed lines of the file:
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@@
 			)
 		)
-		(property "Value" "270k"
+		(property "Value" "100k"
 			(at 180.34 73.6599 0)
 			(effects
